Commit message: Added camera

File: urdf/suii.urdf (robot description, URDF)
Before this commit: robot suii, 18 links, 17 joints
Links:
- added link camera_placeholder, mass 0.001; collision box size=0.005 0.005 0.005; visual box size=0.005 0.005 0.005
Joints:
- added joint camera_joint: type fixed, parent ur3/tool0, child camera_placeholder, origin xyz=0 -0.044877 0.105 rpy=0 -1.57079632679 1.57079632679

Commit message: Added navigation and mapping

File: urdf/suii.urdf (robot description, URDF)
Before this commit: robot suii, 19 links, 18 joints
Links:
- link base_link: mass 31.4408606561222 -> 100
