Commit message: Added table workstations

File: urdf/table.urdf.xacro (robot description, xacro)
@@ -1,13 +1,12 @@
 <?xml version="1.0"?>
 <robot xmlns:xacro="http://www.ros.org/wiki/xacro" name="table">
-<!--<xacro:arg name="height" default="0.05"/>-->
 <link name="base_link">
     <inertial>
-      <origin rpy="0 0 0" xyz="0 0 0"/>
+      <origin rpy="0 0 0" xyz="0 0 ${0.5* $(arg height)}"/>
       <mass value="100"/>
       <inertia ixx="1" ixy="0" ixz="0" iyy="1" iyz="0" izz="1"/>
     </inertial>
     <visual>
-      <origin rpy="0 0 0" xyz="0 0 0"/>
+      <origin rpy="0 0 0" xyz="0 0 ${0.5* $(arg height)}"/>
       <geometry>
         <box size="0.5 0.8 $(arg height)" />
@@ -18,5 +17,5 @@
     </visual>
     <collision>
-      <origin rpy="0 0 0" xyz="0 0 0"/>
+      <origin rpy="0 0 0" xyz="0 0 ${0.5* $(arg height)}"/>
       <geometry>
         <box size="0.5 0.8 $(arg height)" />
@@ -26,4 +25,5 @@
 <gazebo reference="base_link">
     <static>true</static>
+    <kinematic>true</kinematic>
 </gazebo>
 </robot>
